File: Minuteur.kicad_pcb (KiCad board)
At the start: 2 copper layers, 149.9 x 49.5 mm, 46 parts, among them J1 ICSP, J2 Piezo, J3 CONN_01X07, J4 Data, J5 Screw_Terminal_1x03, J6 USB_OTG, J7 Screw_Terminal_1x02, Q1 BC818-40, SW1 SW_Push_SPDT_2Leds, SW2 SW_Push_SPDT_2Leds, SW3 Rotary_Encoder_Switch, U1 MAX7219, U2 ATMEGA8-16AU, U3 PC817, U4 LD1117S50TR, Y1 16MHz

Commit message: v0.9 ready for fab.
Connections:
- SW3 pad 6: (no net) -> GND
Routing:
- net GND: track 168.2 -> 188.8 mm, vias 24 -> 27
- net (no net): track 20.6 -> 0.00 mm, vias 3 -> 0
- net +5V: track 288.5 -> 285.8 mm

Commit message: Preparing v1 fab launch.
Parts:
- removed the U2 at (139.7, 113.0)
- added J8: Outputs, Pin_Headers:Pin_Header_Straight_1x04_Pitch2.54mm, F.Cu at (176.5, 120.7)
- added U1: ATMEGA328P-AU, Housings_QFP:TQFP-32_7x7mm_Pitch0.8mm, F.Cu at (139.7, 113.0)
- J4: renamed from J3; value CONN_01X07 -> Inputs
- RL1: moved to B.Cu
- moved C1 2.87 mm to (130.4, 111.6), turned to 270 degrees
- moved REF** 1.17 mm to (120.9, 117.6)
- moved RL1 0.34 mm to (192.1, 107.9)
- renumbered C3 to C2, C4 to C3, C5 to C4, C2 to C5, D4 to D2, D2 to D3, D3 to D4, J7 to J2, J2 to J3, J4 to J5, J5 to J7, R8 to R1, R11 to R10, R5 to R11, R6 to R12, R1 to R2, R12 to R3, R3 to R4, R7 to R5, R2 to R6, R4 to R7, R9 to R8, R10 to R9, SW3 to SW1, SW1 to SW2, SW2 to SW3, U4 to U2, U1 to U3, U3 to U4
Connections:
- net OUT renamed OUT_1
- D4 pad 2: Net-(D3-Pad2) (its old number) -> Net-(D4-Pad2)
- J3 pad 2: GND -> PIEZO_2
- J7 pad 1: Net-(J5-Pad1) -> Net-(J7-Pad1)
- J7 pad 3: Net-(J5-Pad3) -> Net-(J7-Pad3)
- Q1 pad 3: Net-(D3-Pad2) (its old number) -> Net-(D4-Pad2)
- R1 pad 2: PIEZO -> PIEZO_1
- RL1 pad 2: Net-(D3-Pad2) (its old number) -> +5V
- RL1 pad 3: Net-(J5-Pad1) -> Net-(J7-Pad3)
- RL1 pad 4: Net-(J5-Pad3) -> Net-(J7-Pad1)
- RL1 pad 5: +5V -> Net-(D4-Pad2)
Routing:
- net OUT_2: track 0.00 -> 44.6 mm
- net Net-(D4-Pad2): track 0.00 -> 22.2 mm
- net Net-(D3-Pad2) (its old number): track 21.7 -> 0.00 mm
- net Net-(J5-Pad1): track 18.2 -> 0.00 mm
- net Net-(J5-Pad3): track 18.1 -> 0.00 mm
- net OUT_1: track 72.4 -> 54.6 mm, vias 4 -> 1
- net Net-(J7-Pad3): track 0.00 -> 17.6 mm
- net Net-(J7-Pad1): track 0.00 -> 17.4 mm
- net PIEZO_2: track 0.00 -> 13.9 mm
- net BTN_2: track 100.6 -> 89.5 mm, vias 4 -> 3
- net +5V: track 285.8 -> 292.7 mm
- net RESET: track 37.4 -> 33.5 mm
- net GND: track 188.8 -> 192.6 mm, vias 27 -> 24
- net PIEZO_1: track 0.00 -> 3.77 mm
- net PIEZO: track 3.77 -> 0.00 mm
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Other:
- board text added: "Minuteur v1"
- board text added: "O1"
- board text added: "O2"
- board text added: "https://www.lelabodutroisieme.fr 09/2017"
- board text removed: "Minuteur v0.9"
- board text removed: "https://www.lelabodutroisieme.fr 06/2017"
