File: Minuteur.sch (KiCad schematic (older format))
At the start: 39 parts, among them J1 ICSP, J2 Piezo, J3 CONN_01X07, J4 Data, J5 Screw_Terminal_1x03, J6 USB_OTG, J7 Screw_Terminal_1x02, Q1 BC818-40, SW1 SW_Push_SPDT_2Leds, SW2 SW_Push_SPDT_2Leds, SW3 Rotary_Encoder_Switch, U1 MAX7219, U2 ATMEGA8-16AU, U3 PC817, U4 LD1117S50TR, Y1 16MHz

Commit message: Preparing v1 fab launch.
Parts:
- removed U2: ATMEGA8-16AU, Housings_QFP:TQFP-32_7x7mm_Pitch0.8mm, symbol ATMEGA8-16AU
- added J8: Outputs, Pin_Headers:Pin_Header_Straight_1x04_Pitch2.54mm, symbol Conn_01x04
- added U1: ATMEGA328P-AU, Housings_QFP:TQFP-32_7x7mm_Pitch0.8mm, symbol ATMEGA328P-AU
- J4: renamed from J3; value CONN_01X07 -> Inputs
- renumbered C3 to C2, C4 to C3, C5 to C4, C2 to C5, D4 to D2, D2 to D3, D3 to D4, J7 to J2, J2 to J3, J4 to J5, J5 to J7, R8 to R1, R11 to R10, R5 to R11, R6 to R12, R1 to R2, R12 to R3, R3 to R4, R7 to R5, R2 to R6, R4 to R7, R9 to R8, R10 to R9, SW3 to SW1, SW1 to SW2, SW2 to SW3, U4 to U2, U1 to U3, U3 to U4
Connections:
- net labels added: OUT_1, OUT_2, PIEZO_1, PIEZO_2
- net labels removed: OUT, PIEZO
- wire segments 116 -> 126
- no-connect marks 23 -> 21
Other:
- moved on the sheet: C2, C3, C4, D1, D2, J1, J2, J3, J6, R1, R2, R3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
